Commit message: add ros2 control

File: install/arm_desc/share/arm_desc/urdf/arm.urdf.xacro (robot description, xacro)
@@ -6,5 +6,5 @@
 <xacro:property name="PI" value="3.14159" />
 <xacro:property name="effort" value="30.0" />
-<xacro:property name=" velocity" value="10.0" />
+<xacro:property name="velocity" value="10.0" />
 <xacro:macro name="default_inertia" params="mass">
   <inertial>

File: install/arm_desc/share/arm_desc/urdf/arm_gazebo.xacro (robot description, xacro)
@@ -1,15 +1,16 @@
 <?xml version="1.0"?>
-<robot xmlns:xacro="https://www.ros.org/wiki/xacro" name="arm">
+<robot xmlns:xacro="http://www.ros.org/wiki/xacro" name="arm">
+    <xacro:arg name="is_ignition" default="true"/>
     <gazebo>
-            <xacro:if value="${arg is_ignition}">
-                    <plugin filename="ign_ros2_control-system" name="ign_ros2_control::IgnitionROS2ControlPlugin">
-                            <parameters>$(find arm_controller)/config/arm_controllers.yaml</parameters>
-                    </plugin>
-            </xacro:if>
-            <xacro:unless value="${arg is_ignition}">
-                    <plugin filename="gz_ros2_control_system" name="gz_ros2_control::GazeboROS2ControlPlugin">
-                            <parameters>$(find arm_controller)/config/arm_controllers.yaml</parameters>
-                    </plugin>
-            </xacro:unless>
+        <xacro:if value="$(arg is_ignition)">
+            <plugin filename="ign_ros2_control-system" name="ign_ros2_control::IgnitionROS2ControlPlugin">
+                <parameters>$(find arm_controller)/config/arm_controllers.yaml</parameters>
+            </plugin>
+        </xacro:if>
+        <xacro:unless value="$(arg is_ignition)">
+            <plugin filename="gz_ros2_control-system" name="gz_ros2_control::GazeboROS2ControlPlugin">
+                <parameters>$(find arm_controller)/config/arm_controllers.yaml</parameters>
+            </plugin>
+        </xacro:unless>
     </gazebo>
 </robot>

File: install/arm_desc/share/arm_desc/urdf/arm_ros2_control.xacro (robot description, xacro)
@@ -2,19 +2,23 @@
 <robot xmlns:xacro="https://www.ros.org/wiki/xacro" name="arm">
 <xacro:property name="PI" value="3.14159" />
-        <ros2_control type="system" name="RobotSystem">
-                <xacro:if value="${arg is_ignition}">
-                        <hardware>
-                                <plugin>ign_ros2_control/IgnitionSystem</plugin>
-                        </hardware>
-                </xacro:if>
-                <xacro:unless value="${arg is_ignition}">
-                        <hardware>
-                                <plugin>gz_ros2_control/GazeboSimSystem</plugin>
-                        </hardware>
-                </xacro:unless>
+        <ros2_control name="RobotSystem" type="system">
+        <xacro:property name="PI" value="3.14159265359" />
+        <!-- ros2_control Gazebo -->
+        <!-- ROS 2 Humble -->
+        <xacro:if value="$(arg is_ignition)">
+            <hardware>
+                <plugin>ign_ros2_control/IgnitionSystem</plugin>
+            </hardware>
+        </xacro:if>
+        <!-- ROS 2 Iron or above -->
+        <xacro:unless value="$(arg is_ignition)">
+            <hardware>
+                <plugin>gz_ros2_control/GazeboSimSystem</plugin>
+            </hardware>
+        </xacro:unless>
         <joint name="joint_1">
             <command_interface name="position">
-                    <param name="min">${PI/2}</param>
-                    <param name="max">${PI/2}</param>
+            <param name="min">-${PI / 2}</param>
+            <param name="max">${PI / 2}</param>
             </command_interface>
             <state_interface name="position"/>
@@ -22,6 +26,6 @@
         <joint name="joint_2">
             <command_interface name="position">
-                    <param name="min">${PI/2}</param>
-                    <param name="max">${PI/2}</param>
+            <param name="min">-${PI / 2}</param>
+            <param name="max">${PI / 2}</param>
             </command_interface>
             <state_interface name="position"/>
@@ -29,6 +33,6 @@
         <joint name="joint_3">
             <command_interface name="position">
-                    <param name="min">${PI/2}</param>
-                    <param name="max">${PI/2}</param>
+            <param name="min">-${PI / 2}</param>
+            <param name="max">${PI / 2}</param>
             </command_interface>
             <state_interface name="position"/>
@@ -36,12 +40,12 @@
         <joint name="joint_4">
             <command_interface name="position">
-                    <param name="min">${PI/2}</param>
-                    <param name="max">0.0</param>
+            <param name="min">-${PI / 2}</param>
+            <param name="max">0.0</param>
             </command_interface>
             <state_interface name="position"/>
         </joint>
         <joint name="joint_5">
-                <param name="mimic">joint_4</param>
-                <param name="multiplier">-1</param>
+            <param name="mimic">joint_4</param>
+            <param name="multiplier">-1</param>
         </joint>
         </ros2_control>
